File: TempSense.kicad_pcb (KiCad board)
At the start: 2 copper layers, 40 x 21.8 mm, 32 parts, among them J1 Conn_01x02_Pin, P1 USB_C_Plug_USB2.0, U1 MCP73831-2-OT, U2 BME680, U3 AP2112K-3.3, U4 ESP32-C6-MINI-1

Commit message: stuffs
Parts:
- added C13: 1uF, Capacitor_SMD:C_0402_1005Metric, F.Cu at (164.9, 75.3)
- added R9: 10k, Resistor_SMD:R_0402_1005Metric, F.Cu at (172.1, 73.5)
- added SW1: SW_Push, Button_Switch_SMD:SW_Push_SPST_NO_Alps_SKRK, F.Cu at (168.7, 75.0)
- added SW2: SW_Push, Button_Switch_SMD:SW_Push_SPST_NO_Alps_SKRK, F.Cu at (173.6, 88.8)
Connections:
- U4 pad 23: unconnected-(U4-IO9-Pad23) -> /boot
Routing:
- net /boot: track 0.00 -> 8.14 mm
- net /EN: track 0.00 -> 7.35 mm
- net GND: track 31.9 -> 33.7 mm, vias 9 -> 17
- net Net-(C13-Pad1): track 0.00 -> 1.31 mm
Other:
- board size 40 x 21.8 mm -> 40 x 22.1 mm
