File: TempSense.kicad_pcb (KiCad board)
At the start: 2 copper layers, 40 x 22.1 mm, 38 parts, among them J1 Conn_01x02_Pin, P1 USB_C_Plug_USB2.0, SW1 SW_Push, SW2 SW_Push, U1 MCP73831-2-OT, U2 BME680, U3 AP2112K-3.3, U4 ESP32-C6-MINI-1

Commit message: almost finished
Parts:
- added C15: 1uF, Capacitor_SMD:C_0402_1005Metric, F.Cu at (168.8, 81.0)
- added C16: 100nf, Capacitor_SMD:C_0402_1005Metric, F.Cu at (182.9, 74.5)
- added G***: LOGO, LOGO, B.Cu at (166.0, 79.3)
- added U5: TSL25911FN, OptoDevice:AMS_TSL25911FN, F.Cu at (166.5, 81.0)
- moved C6 24.5 mm to (160.4, 84.2), turned to 0 degrees
- moved C5 2.38 mm to (168.6, 85.6)
- moved C7 1.91 mm to (162.3, 84.2)
- moved C14 0.49 mm to (170.6, 85.6)
Connections:
- net /BAT+ renamed +BATT
- R3 pad 1: /SCL-BME680 -> /SCL
- R4 pad 1: /SDA-BME680 -> /SDA
- U2 pad 3: /SDA-BME680 -> /SDA
- U2 pad 4: /SCL-BME680 -> /SCL
- U4 pad 15: unconnected-(U4-IO6-Pad15) -> /SDA
- U4 pad 16: /SDA-BME680 -> /SCL
- U4 pad 22: /SCL-BME680 -> unconnected-(U4-IO8-Pad22)
- U4 pad 24: unconnected-(U4-IO18-Pad24) -> /IO18
- U4 pad 25: unconnected-(U4-IO19-Pad25) -> /IO19
- U4 pad 26: unconnected-(U4-IO20-Pad26) -> /IO20
- U4 pad 27: unconnected-(U4-IO21-Pad27) -> /IO21
- U4 pad 28: unconnected-(U4-IO22-Pad28) -> /IO22
Routing:
- net /SDA: track 0.00 -> 35.0 mm, vias 0 -> 3
- net /SDA-BME680: track 31.8 -> 0.00 mm, vias 2 -> 0
- net /SCL-BME680: track 31.4 -> 0.00 mm, vias 2 -> 0
- net /SCL: track 0.00 -> 29.0 mm, vias 0 -> 2
- net +3V3: track 102.5 -> 107.0 mm
- net +BATT: track 20.9 -> 19.3 mm
- net GND: track 52.9 -> 51.3 mm, vias 22 -> 24
- net /LED: track 13.0 -> 11.7 mm
- net Net-(P1-D+): track 20.2 -> 20.9 mm
Other:
- outline, holes or cut-outs redrawn
