File: TempSense.kicad_sch (KiCad schematic)
At the start: 34 parts, among them J1 Conn_01x02_Pin, P1 USB_C_Plug_USB2.0, SW1 SW_Push, SW2 SW_Push, U1 MCP73831-2-OT, U2 BME680, U3 AP2112K-3.3, U4 ESP32-C6-MINI-1

Commit message: stuffs
Parts:
- added C13: 1uF, Capacitor_SMD:C_0402_1005Metric, symbol Device:C
- added R9: 10k, Resistor_SMD:R_0402_1005Metric, symbol Device:R
- SW1, SW2: footprint (none) -> Button_Switch_SMD:SW_Push_SPST_NO_Alps_SKRK
Connections:
- net +3V3: now also R9.1
- net EN: now also SW1.2, R9.2
- net GND: now also SW2.1, C13.2
- net at SW1.1: now also C13.1
- net boot: now reaches SW2.2
- net boot: now also U4.23 (IO9)
Other:
- moved on the sheet: C1, C10, C11, C12, C2, C3, C4, C5, C6, C7, C8, C9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
