File: TempSense.kicad_sch (KiCad schematic)
At the start: 43 parts, among them J1 Conn_01x02_Pin, P1 USB_C_Plug_USB2.0, SW1 SW_Push, SW2 SW_Push, U1 MCP73831-2-OT, U2 BME680, U3 AP2112K-3.3, U4 ESP32-C6-MINI-1

Commit message: almost finished
Parts:
- added C15: 1uF, Capacitor_SMD:C_0402_1005Metric, symbol Device:C
- added C16: 100nf, Capacitor_SMD:C_0402_1005Metric, symbol Device:C_Small
- added U5: TSL25911FN, OptoDevice:AMS_TSL25911FN, symbol Sensor_Optical:TSL25911FN
Connections:
- net EN is gone; now on net +3V3: C13.1, R9.2, SW1.2, U4.8 (EN)
- net +3V3: now also C15.1, C16.1, U5.5 (VDD)
- net GND: now also C15.2, C16.2, U5.3 (GND)
- net SDA: now reaches U4.15 (IO6)
- net SDA: now also R4.1, U2.3 (SDI), U5.6 (SDA)
- net SCL-BME680 renamed SCL
- net SCL: now also U4.16 (IO7), U5.1 (SCL); no longer U4.22 (IO8)
- removed net SDA-BME680: R4.1, U2.3 (SDI), U4.16 (IO7)
- no-connect marks 1 -> 11
Other:
- moved on the sheet: C1, C10, C11, C12, C13, C14, C2, C3, C4, C5, C6, C7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
