File: kaze.kicad_pcb (KiCad board)
At the start: 2 copper layers, 40 x 22.1 mm, 50 parts, among them J1 Conn_01x02_Pin, P1 USB_C_Plug_USB2.0, SW1 SW_Push, SW2 SW_Push, U1 MCP73831-2-OT, U2 BME680, U3 AP2112K-3.3, U4 ESP32-C6-MINI-1, U5 TSL25911FN, U6 SGP40-D-R4

Commit message: pcb stuff
Parts:
- removed the C17 at (169.6, 75.9)
- removed C18: 1uF, Capacitor_SMD:C_0402_1005Metric
- removed IO2, IO3: TestPoint, TestPoint:TestPoint_Pad_D3.0mm
- removed the R11 at (164.2, 75.1)
- removed the R9 at (177.1, 73.5)
- removed U6: SGP40-D-R4, SGP40_D_R4:XCDR_SGP40-D-R4
- C1: renamed from C2; value 100nf -> 100nF
- C10: renamed from C16; value 100nf -> 100nF
- C11: renamed from C1; value 4.7u -> 4.7uF
- C12: renamed from C8; value 100nf -> 100nF
- C13: renamed from C9; value 100nf -> 100nF
- C14: renamed from C10; value 100nf -> 100nF
- C15: renamed from C11; value 100nf -> 100nF
- C16: renamed from C12; value 100nf -> 100nF
- C17: renamed from C4; value 4.7u -> 4.7uF
- C2: renamed from C3; value 100nf -> 100nF
- C6: renamed from C5; value 10uf -> 10uF
- C7: renamed from C6; value 10u -> 10uF
- C8: renamed from C7; value 100n -> 100nF
- renumbered C13 to C3, C15 to C4, C14 to C5, C19 to C9, R12 to R10, R7 to R11, R9 to R3, R5 to R4, R6 to R5, R10 to R6, R8 to R7, R4 to R8, R3 to R9, U5 to U1, U1 to U5
Connections:
- P1 pad A6: Net-(P1-D+) -> Net-(P1-D+-PadA6)
- P1 pad A7: Net-(P1-D-) -> Net-(P1-D--PadA7)
- P1 pad A8: (no net) -> GND
- P1 pad B6: (no net) -> Net-(P1-D+-PadA6)
- P1 pad B7: (no net) -> Net-(P1-D--PadA7)
- P1 pad B8: (no net) -> GND
- R4 pad 1: Net-(P1-D-) -> Net-(P1-D--PadA7)
- R5 pad 1: Net-(P1-D+) -> Net-(P1-D+-PadA6)
Routing:
- net /SCL: track 41.2 -> 29.0 mm, vias 4 -> 2
- net +3V3: track 121.2 -> 111.7 mm, vias 5 -> 3
- net /IO2: track 8.79 -> 0.00 mm, vias 1 -> 0
- net /IO3: track 6.81 -> 0.00 mm, vias 1 -> 0
- net Net-(P1-D+-PadA6): track 0.00 -> 6.53 mm, vias 0 -> 2
- net /SDA: track 40.5 -> 35.0 mm, vias 4 -> 3
- net GND: track 60.9 -> 56.4 mm, vias 31 -> 29
- net Net-(P1-D--PadA7): track 0.00 -> 4.20 mm
- net Net-(U6-VDD): track 2.09 -> 0.00 mm
- net Net-(P1-D-): track 1.76 -> 0.00 mm
- net Net-(P1-D+): track 1.64 -> 0.00 mm
- net +5V: track 16.9 -> 17.7 mm
- net /EN: track 6.83 -> 6.23 mm
Other:
- outline, holes or cut-outs redrawn
- board text added: "kaze - v0 - 2026"
- board text removed: "(kaze)"
