File: kaze.kicad_sch (KiCad schematic)
At the start: 46 parts, among them J1 Conn_01x02_Pin, P1 USB_C_Plug_USB2.0, SW1 SW_Push, SW2 SW_Push, U1 MCP73831-2-OT, U2 BME680, U3 AP2112K-3.3, U4 ESP32-C6-MINI-1, U5 TSL25911FN

Commit message: pcb
Parts:
- removed D6: SS14, Diode_SMD:D_SMA, symbol Diode:SS14
- added C17, C18: 1uF, Capacitor_SMD:C_0402_1005Metric, symbol Device:C
- added C19: 22uf, Capacitor_SMD:C_0402_1005Metric, symbol Device:C_Small
- added R11: 4.7, Resistor_SMD:R_0402_1005Metric, symbol Device:R
- added R12: 10k, Resistor_SMD:R_0402_1005Metric, symbol Device:R_Small
- added U6: SGP40-D-R4, SGP40_D_R4:XCDR_SGP40-D-R4, symbol SGP40-D-R4:SGP40-D-R4
- C13: value 10uF -> 1uF
Connections:
- net +3V3: now also C17.1, C19.1, R11.2, R12.1, U6.5 (VDDH); no longer C13.1, R9.2, SW1.2, U4.8 (EN)
- net +BATT: now also U3.1 (VIN), U3.3 (EN)
- net GND: now also C17.2, C18.2, C19.2, U6.2 (VSS), U6.4 (N/A), U6.7 (EXP)
- net SCL: now also U6.6 (SCL)
- net SDA: now also U6.3 (SDA)
- net at U4.22 (IO8): now also R12.2
- new net: C18.1, R11.1, U6.1 (VDD)
- new net EN: C13.1, R9.2, SW1.2, U4.8 (EN)
Other:
- moved on the sheet: C10, C11, C12, C8, C9, D1, D2, D3, D4, D5, TP1, TP2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
