File: kaze.kicad_sch (KiCad schematic)
At the start: 48 parts, among them J1 Conn_01x02_Pin, P1 USB_C_Plug_USB2.0, SW1 SW_Push, SW2 SW_Push, U1 MCP73831-2-OT, U2 BME680, U3 AP2112K-3.3, U4 ESP32-C6-MINI-1, U5 TSL25911FN, U6 SGP40-D-R4

Commit message: pcb stuff
Parts:
- removed C17, C18: 1uF, Capacitor_SMD:C_0402_1005Metric, symbol Device:C
- removed R11: 4.7, Resistor_SMD:R_0402_1005Metric, symbol Device:R
- removed TP1, TP2: TestPoint, TestPoint:TestPoint_Pad_D3.0mm, symbol Connector:TestPoint
- removed U6: SGP40-D-R4, SGP40_D_R4:XCDR_SGP40-D-R4, symbol SGP40-D-R4:SGP40-D-R4
- C1: renamed from C2; value 100nf -> 100nF
- C10: renamed from C16; value 100nf -> 100nF
- C11: renamed from C1; value 4.7u -> 4.7uF
- C12: renamed from C8; value 100nf -> 100nF
- C13: renamed from C9; value 100nf -> 100nF
- C14: renamed from C10; value 100nf -> 100nF
- C15: renamed from C11; value 100nf -> 100nF
- C16: renamed from C12; value 100nf -> 100nF
- C17: renamed from C4; value 4.7u -> 4.7uF
- C2: renamed from C3; value 100nf -> 100nF
- C6: renamed from C5; value 10uf -> 10uF
- C7: renamed from C6; value 10u -> 10uF
- C8: renamed from C7; value 100n -> 100nF
- P1: symbol Connector:USB_C_Plug_USB2.0 -> Connector:USB_C_Receptacle_USB2.0_16P
- renumbered C13 to C3, C15 to C4, C14 to C5, C19 to C9, R12 to R10, R7 to R11, R9 to R3, R5 to R4, R6 to R5, R10 to R6, R8 to R7, R4 to R8, R3 to R9, U5 to U1, U1 to U5
Connections:
- net GND: now also P1.A8 (SBU1), P1.B8 (SBU2)
- net at P1.A6 (D+), R5.1: now also P1.B6 (D+)
- net at P1.A7 (D-), R4.1: now also P1.B7 (D-)
Other:
- moved on the sheet: J1
