File: pcb/kaze.kicad_pcb (KiCad board)
At the start: 2 copper layers, 40 x 22.1 mm, 43 parts, among them J1 Conn_01x02_Pin, P1 USB_C_Plug_USB2.0, SW1 SW_Push, SW2 SW_Push, U1 TSL25911FN, U2 BME680, U3 AP2112K-3.3, U4 ESP32-C6-MINI-1, U5 MCP73831-2-OT

Commit message: update
Parts:
- added J2: Conn_02x02_Odd_Even, Connector_PinHeader_1.00mm:PinHeader_2x02_P1.00mm_Vertical, F.Cu at (169.4, 75.1)
- J1: footprint Connector_PinHeader_1.00mm:PinHeader_2x01_P1.00mm_Vertical -> Connector_PinHeader_1.00mm:PinHeader_1x02_P1.00mm_Vertical; moved to B.Cu
- moved J1 0.76 mm to (163.3, 88.5), turned to 180 degrees
- moved R3 0.54 mm to (176.7, 74.5)
- moved C3 0.50 mm to (175.8, 73.5)
Connections:
- U4 pad 10: unconnected-(U4-IO5-Pad10) -> /IO5
- U4 pad 9: unconnected-(U4-IO4-Pad9) -> /IO4
Routing:
- net /IO2: track 0.00 -> 18.7 mm, vias 0 -> 1
- net /IO3: track 0.00 -> 15.5 mm, vias 0 -> 1
- net /IO4: track 0.00 -> 8.57 mm, vias 0 -> 1
- net /IO5: track 0.00 -> 7.54 mm
- net GND: track 56.4 -> 60.3 mm
- net +3V3: track 111.7 -> 110.6 mm
