File: pcb/kaze.kicad_sch (KiCad schematic)
At the start: 42 parts, among them J1 Conn_01x02_Pin, P1 USB_C_Plug_USB2.0, SW1 SW_Push, SW2 SW_Push, U1 TSL25911FN, U2 BME680, U3 AP2112K-3.3, U4 ESP32-C6-MINI-1, U5 MCP73831-2-OT

Commit message: update
Parts:
- added J2: Conn_02x02_Odd_Even, Connector_PinHeader_1.00mm:PinHeader_2x02_P1.00mm_Vertical, symbol Connector_Generic:Conn_02x02_Odd_Even
- J1: footprint Connector_PinHeader_1.00mm:PinHeader_2x01_P1.00mm_Vertical -> Connector_PinHeader_1.00mm:PinHeader_1x02_P1.00mm_Vertical
Connections:
- net IO2: now also J2.1 (Pin_1)
- net IO3: now also J2.2 (Pin_2)
- net IO5: now reaches U4.10 (IO5)
- net IO5: now also J2.4 (Pin_4)
- net IO4: now reaches U4.9 (IO4)
- net IO4: now also J2.3 (Pin_3)
- no-connect marks 14 -> 12
Changed lines of the file:
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@@
 	)
 	(no_connect
-		(at 100.33 111.76)
-	)
-	(no_connect
-		(at 100.33 114.3)
-	)
-	(no_connect
 		(at 264.16 133.35)
 	)
@@
 	(wire
 		(pts
+			(xy 231.14 68.58) (xy 240.03 68.58)
+		)
+		(stroke
+			(width 0)
+			(type default)
+		)
+	)
+	(wire
+		(pts
 			(xy 21.59 81.28) (xy 31.75 81.28)
 		)
@@
 	(wire
 		(pts
+			(xy 231.14 66.04) (xy 240.03 66.04)
+		)
+		(stroke
+			(width 0)
+			(type default)
+		)
+	)
+	(wire
+		(pts
 			(xy 33.02 83.82) (xy 31.75 83.82)
 		)
@@
 	(wire
 		(pts
+			(xy 91.44 111.76) (xy 91.44 110.49)
+		)
+		(stroke
+			(width 0)
+			(type default)
+		)
+	)
+	(wire
+		(pts
 			(xy 237.49 142.24) (xy 237.49 144.78)
 		)
@@
 	(wire
 		(pts
+			(xy 85.09 111.76) (xy 88.9 111.76)
+		)
+		(stroke
+			(width 0)
+			(type default)
+		)
+	)
+	(wire
+		(pts
 			(xy 41.91 53.34) (xy 41.91 62.23)
 		)
@@
 	(wire
 		(pts
+			(xy 100.33 111.76) (xy 91.44 111.76)
+		)
+		(stroke
+			(width 0)
+			(type default)
+		)
+	)
+	(wire
+		(pts
 			(xy 172.72 60.96) (xy 172.72 62.23)
 		)
@@
 	(wire
 		(pts
+			(xy 260.35 66.04) (xy 252.73 66.04)
+		)
+		(stroke
+			(width 0)
+			(type default)
+		)
+	)
+	(wire
+		(pts
 			(xy 41.91 62.23) (xy 26.67 62.23)
 		)
@@
 	(wire
 		(pts
+			(xy 91.44 110.49) (xy 88.9 110.49)
+		)
+		(stroke
+			(width 0)
+			(type default)
+		)
+	)
+	(wire
+		(pts
 			(xy 66.04 59.69) (xy 66.04 57.15)
 		)
@@
 	(wire
 		(pts
+			(xy 260.35 68.58) (xy 252.73 68.58)
+		)
+		(stroke
+			(width 0)
+			(type default)
+		)
+	)
+	(wire
+		(pts
 			(xy 187.96 133.35) (xy 191.77 133.35)
 		)
@@
 	(wire
 		(pts
+			(xy 88.9 110.49) (xy 88.9 111.76)
+		)
+		(stroke
+			(width 0)
+			(type default)
+		)
+	)
+	(wire
+		(pts
 			(xy 199.39 118.11) (xy 180.34 118.11)
 		)
@@
 	(wire
 		(pts
+			(xy 85.09 114.3) (xy 100.33 114.3)
+		)
+		(stroke
+			(width 0)
+			(type default)
+		)
+	)
+	(wire
+		(pts
 			(xy 114.3 25.4) (xy 114.3 36.83)
 		)
@@
 		)
 	)
+	(label "IO3"
+		(at 260.35 66.04 180)
+		(effects
+			(font
+				(size 1.27 1.27)
+			)
+			(justify right bottom)
+		)
+	)
+	(label "IO2"
+		(at 231.14 66.04 0)
+		(effects
+			(font
+				(size 1.27 1.27)
+			)
+			(justify left bottom)
+		)
+	)
 	(label "STAT"
 		(at 54.61 123.19 180)
@@
 		)
 	)
+	(label "IO5"
+		(at 260.35 68.58 180)
+		(effects
+			(font
+				(size 1.27 1.27)
+			)
+			(justify right bottom)
+		)
+	)
 	(label "D-"
 		(at 59.69 35.56 180)
@@
 		)
 	)
+	(label "IO4"
+		(at 85.09 111.76 0)
+		(effects
+			(font
+				(size 1.27 1.27)
+			)
+			(justify left bottom)
+		)
+	)
 	(label "IO2"
 		(at 85.09 106.68 0)
@@
 		)
 	)
+	(label "IO4"
+		(at 231.14 68.58 0)
+		(effects
+			(font
+				(size 1.27 1.27)
+			)
+			(justify left bottom)
+		)
+	)
 	(label "EN"
 		(at 92.71 96.52 0)
@@
 		)
 	)
+	(label "IO5"
+		(at 85.09 114.3 0)
+		(effects
+			(font
+				(size 1.27 1.27)
+			)
+			(justify left bottom)
+		)
+	)
 	(label "STAT"
 		(at 80.01 101.6 0)
@@
 	)
 	(symbol
+		(lib_id "Connector_Generic:Conn_02x02_Odd_Even")
+		(at 245.11 66.04 0)
+		(unit 1)
+		(exclude_from_sim no)
+		(in_bom yes)
+		(on_board yes)
+		(dnp no)
+		(fields_autoplaced yes)
+		(property "Reference" "J2"
+			(at 246.38 59.69 0)
+			(effects
+				(font
+					(size 1.27 1.27)
+				)
+			)
+		)
+		(property "Value" "Conn_02x02_Odd_Even"
+			(at 246.38 62.23 0)
+			(effects
+				(font
+					(size 1.27 1.27)
+				)
+			)
+		)
+		(property "Footprint" "Connector_PinHeader_1.00mm:PinHeader_2x02_P1.00mm_Vertical"
+			(at 245.11 66.04 0)
+			(effects
+				(font
+					(size 1.27 1.27)
+				)
+				(hide yes)
+			)
+		)
+		(property "Datasheet" "~"
+			(at 245.11 66.04 0)
+			(effects
+				(font
+					(size 1.27 1.27)
+				)
+				(hide yes)
+			)
+		)
+		(property "Description" "Generic connector, double row, 02x02, odd/even pin numbering scheme (row 1 odd numbers, row 2 even numbers), script generated (kicad-library-utils/schlib/autogen/connector/)"
+			(at 245.11 66.04 0)
+			(effects
+				(font
+					(size 1.27 1.27)
+				)
+				(hide yes)
+			)
+		)
+		(pin "2"
+		)
+		(pin "3"
+		)
+		(pin "1"
+		)
+		(pin "4"
+		)
+		(instances
+			(project ""
+				(path "/f63e4aaa-0236-48be-b6f2-3deed72e8a67"
+					(reference "J2")
+					(unit 1)
+				)
+			)
+		)
+	)
+	(symbol
 		(lib_id "Device:C")
 		(at 262.89 31.75 0)
@@
 			)
 		)
-		(property "Footprint" "Connector_PinHeader_1.00mm:PinHeader_2x01_P1.00mm_Vertical"
+		(property "Footprint" "Connector_PinHeader_1.00mm:PinHeader_1x02_P1.00mm_Vertical"
 			(at 55.88 59.69 0)
 			(effects
